File: Hardware/USBussy_Current_Probe.kicad_sch (KiCad schematic)
At the start: 29 parts, among them J2 Mobo header, J3 CFG_OPT1, J4 CFG_COM, J5 CFG_OPT2, J6 USB_A, J7 Jumper holder, J8 MEAS, Q1 RE1C002UN, Q2 RE1C002UN, U1 AP2151W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

Commit message: Add texts on board and export
Parts:
- added SYM1: ~, leptunKicadLib:AMOGUS, symbol Graphic:Logo_Open_Hardware_Small
Changed lines of the file:
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@@
+    )
+  )
+  (symbol (lib_id "Graphic:Logo_Open_Hardware_Small") (at 17.78 17.78 0) (unit 1)
+    (in_bom no) (on_board yes) (dnp no) (fields_autoplaced)
+    (property "Reference" "SYM1" (at 17.78 10.795 0)
+      (effects (font (size 1.27 1.27)) hide)
+    )
+    (property "Value" "~" (at 17.78 23.495 0)
+      (effects (font (size 1.27 1.27)) hide)
+    )
+    (property "Footprint" "leptunKicadLib:AMOGUS" (at 17.78 17.78 0)
+      (effects (font (size 1.27 1.27)) hide)
+    )
+    (property "Datasheet" "~" (at 17.78 17.78 0)
+      (effects (font (size 1.27 1.27)) hide)
+    )
+    (property "Sim.Enable" "0" (at 17.78 17.78 0)
+      (effects (font (size 1.27 1.27)) hide)
+    )
+    (instances
+      (project "USBussy_Current_Probe"
+        (path "/bd78fd95-da96-465b-ba6a-93d3623f5005"
+          (reference "SYM1") (unit 1)
+        )
+      )
+      (project "Avionus_Flight_Controller"
+        (path "/ddc7e940-0588-4587-8902-8ced9e615ace"
+          (reference "SYM101") (unit 1)
+        )
+      )
     )
   )
